Commit message: moved main files in the branch

File: jaco_tutorial/jaco_on_table/urdf/jaco_on_table_robot.urdf (robot description, URDF)
Before this commit: robot JacoOnTable, 31 links, 30 joints
Joints:
- joint jaco_finger_joint_0: limit lower=-0.0045 upper=1.05 effort=1.5 velocity=0.2 -> lower=-0.0045 upper=1.05 effort=1.5 velocity=0.3
- joint jaco_finger_joint_2: limit lower=-0.0045 upper=1.05 effort=1.5 velocity=0.2 -> lower=-0.0045 upper=1.05 effort=1.5 velocity=0.3
- joint jaco_finger_joint_4: limit lower=-0.0045 upper=1.05 effort=1.5 velocity=0.2 -> lower=-0.0045 upper=1.05 effort=1.5 velocity=0.3
